Commit message: kinect urdf updated to work with the new dae

File: urdf/kinect.urdf.xacro (robot description, xacro)
@@ -15,5 +15,5 @@
     <link name="${prefix}link">
       <visual>
-        <origin xyz="0 0 0" rpy="0 0 0"/>
+        <origin xyz="0 0 0" rpy="0 0 ${M_PI/2}"/>
         <geometry>
           <mesh filename="package://roboticarts_sensors/meshes/kinect.dae" />
