Commit message: GPU option implemented

File: urdf/rplidar_A1M8.urdf.xacro (robot description, xacro)
@@ -2,5 +2,5 @@
 <robot name="sensor_rplidar_A1M8" xmlns:xacro="http://www.ros.org/wiki/xacro">
 <!-- - - - - - - - - - - - - - RPLIDAR SENSOR - - - - - - - - - - - - - -->
-  <xacro:macro name ="sensor_rplidar_A1M8" params="prefix prefix_topic:='front_laser/scan' use_sim parent *origin">
+  <xacro:macro name ="sensor_rplidar_A1M8" params="prefix prefix_topic:='front_laser/scan' use_sim gpu_sim='false' parent *origin">
     <link name="${prefix}link">
       <collision>
@@ -29,5 +29,5 @@
     </joint>
 		<!-- rplidar A1M8 sensor for simulation -->
-    <xacro:if value="$(arg use_sim)">
+    <xacro:if value="${use_sim}">
       <xacro:sensor_rplidar_A1M8_gazebo/>
     </xacro:if>
@@ -35,6 +35,14 @@
 <!-- - - - - - - - - - - - - - RPLIDAR GAZEBO - - - - - - - - - - - - - -->
   <xacro:macro name="sensor_rplidar_A1M8_gazebo">
+      <xacro:if value="${gpu_sim}">
+        <xacro:property name="ray_type" value="gpu_ray" />
+        <xacro:property name="plugin_filename" value="libgazebo_ros_gpu_laser.so" />
+      </xacro:if>
+      <xacro:unless value="${gpu_sim}">
+        <xacro:property name="ray_type" value="ray" />
+        <xacro:property name="plugin_filename" value="libgazebo_ros_laser.so" />
+    </xacro:unless>
     <gazebo reference="${prefix}link">
-      <sensor type="ray" name="${prefix}sensor">
+      <sensor type="${ray_type}" name="${prefix}sensor">
         <pose>0 0 0 0 0 0</pose>
         <visualize>false</visualize>
@@ -60,5 +68,5 @@
           </noise>
         </ray>
-        <plugin name="${prefix}controller" filename="libgazebo_ros_laser.so">
+        <plugin name="${prefix}controller" filename="${plugin_filename}">
           <topicName>${prefix_topic}</topicName>
           <frameName>/${prefix}link</frameName>

File: urdf/ydlidar_x2.urdf.xacro (robot description, xacro)
@@ -2,5 +2,5 @@
 <robot name="sensor_ydlidar_x2" xmlns:xacro="http://www.ros.org/wiki/xacro">
 <!-- - - - - - - - - - - - - - RPLIDAR SENSOR - - - - - - - - - - - - - -->
-  <xacro:macro name ="sensor_ydlidar_x2" params="prefix prefix_topic:='front_laser/scan' use_sim parent *origin">
+  <xacro:macro name ="sensor_ydlidar_x2" params="prefix prefix_topic:='front_laser/scan' use_sim gpu_sim='false' parent *origin">
     <link name="${prefix}link">
       <collision>
@@ -29,5 +29,5 @@
     </joint>
 		<!-- ydlidar x2 sensor for simulation -->
-    <xacro:if value="$(arg use_sim)">
+    <xacro:if value="${use_sim}">
       <xacro:sensor_ydlidar_x2_gazebo/>
     </xacro:if>
@@ -35,6 +35,14 @@
 <!-- - - - - - - - - - - - - - YDLIDAR GAZEBO - - - - - - - - - - - - - -->
   <xacro:macro name="sensor_ydlidar_x2_gazebo">
+    <xacro:if value="${gpu_sim}">
+        <xacro:property name="ray_type" value="gpu_ray" />
+        <xacro:property name="plugin_filename" value="libgazebo_ros_gpu_laser.so" />
+      </xacro:if>
+      <xacro:unless value="${gpu_sim}">
+        <xacro:property name="ray_type" value="ray" />
+        <xacro:property name="plugin_filename" value="libgazebo_ros_laser.so" />
+    </xacro:unless>
     <gazebo reference="${prefix}link">
-      <sensor type="ray" name="${prefix}sensor">
+      <sensor type="${ray_type}" name="${prefix}sensor">
         <pose>0 0 0 0 0 0</pose>
         <visualize>false</visualize>
@@ -60,5 +68,5 @@
           </noise>
         </ray>
-        <plugin name="${prefix}controller" filename="libgazebo_ros_laser.so">
+        <plugin name="${prefix}controller" filename="${plugin_filename}">
           <topicName>${prefix_topic}</topicName>
           <frameName>/${prefix}link</frameName>
